Commit message: Add effort and velocity limits for rrbot continuous joints

File: play_motion2/test/rrbot/rrbot.xacro (robot description, xacro)
@@ -52,4 +52,5 @@
     <axis xyz="0 1 0"/>
     <dynamics damping="0.7"/>
+    <limit effort="100.0" velocity="1.0"/>
   </joint>
   <!-- Middle Link -->
@@ -83,4 +84,5 @@
     <axis xyz="0 1 0"/>
     <dynamics damping="0.7"/>
+    <limit effort="100.0" velocity="1.0"/>
   </joint>
   <!-- Top Link -->
